Commit message: Add camera

File: src/my_robot/urdf/my_robot.xacro (robot description, xacro)
@@ -117,3 +117,32 @@
     <dynamics damping="1.0" friction="1.0"/>
   </joint>
+  <link name = "camera">
+    <visual>
+      <origin xyz = "0 0 0" rpy = "0 0 0"/>
+      <geometry>
+        <box size = "0.05 0.05 0.05"/>
+      </geometry>
+    </visual>
+    <collision>
+      <origin xyz = "0 0 0" rpy = "0 0 0"/>
+      <geometry>
+        <box size = "0.05 0.05 0.05"/>
+      </geometry>
+    </collision>
+    <inertial>
+      <origin xyz = "0 0 0" rpy = "0 0 0"/>
+      <mass value = "0.1"/>
+      <inertia
+          ixx="1e-6" ixy="0" ixz="0"
+          iyy="1e-6" iyz="0"
+          izz="1e-6"
+      />
+    </inertial>
+  </link>
+  <joint name="camera_joint" type="fixed">
+    <parent link="chassis"/>
+    <child link="camera"/>
+    <axis xyz="0 1 0" rpy="0 0 0"/>
+    <origin xyz="0.2 0 0" rpy="0 0 0"/>
+  </joint>
 </robot>

Commit message: Add lidar

File: src/my_robot/urdf/my_robot.xacro (robot description, xacro)
@@ -143,6 +143,47 @@
     <parent link="chassis"/>
     <child link="camera"/>
-    <axis xyz="0 1 0" rpy="0 0 0"/>
     <origin xyz="0.2 0 0" rpy="0 0 0"/>
+    <axis xyz="0 1 0"/>
   </joint>
+  <link name = "hokuyo">
+    <visual>
+      <origin xyz="0 0 0" rpy="0 0 0"/>
+      <geometry>
+        <mesh filename="package://my_robot/meshes/hokuyo.dae"/>
+      </geometry>
+    </visual>
+    <collision>
+      <origin xyz="0 0 0" rpy="0 0 0"/>
+      <geometry>
+        <box size="0.1 0.1 0.1" />
+      </geometry>
+    </collision>
+    <intertial>
+      <mass value="1e-5"/>
+      <inertia
+        ixx="1e-6" ixy="0" ixz="0"
+        iyy="1e-6" iyz="0"
+        izz="1e-6"
+      />
+    </intertial>
+  </link>
+  <joint name="hokuyo_joint" type="fixed">
+    <parent link="chassis"/>
+    <child link="hokuyo"/>
+    <origin xyz="0.15 0 0.1" rpy="0 0 0"/>
+    <axis xyz="0 1 0"/>
+  </joint>
+  <!-- Add colors -->
+  <gazebo reference="left_wheel">
+    <material>Gazebo/Green</material>
+  </gazebo>
+  <gazebo reference="right_wheel">
+    <material>Gazebo/Green</material>
+  </gazebo>
+  <gazebo reference="chassis">
+    <material>Gazebo/Blue</material>
+  </gazebo>
+  <gazebo reference="camera">
+    <material>Gazebo/Red</material>
+  </gazebo>
 </robot>

Commit message: Add localization

File: src/my_robot/urdf/my_robot.xacro (robot description, xacro)
@@ -56,4 +56,10 @@
     </visual>
   </link>
+  <!-- Macro for calculating cylidner inertia -->
+  <macro name="cylinder_inertia" params="m r h">
+    <inertia  ixx="${m*(3*r*r+h*h)/12}" ixy = "0" ixz = "0"
+              iyy="${m*(3*r*r+h*h)/12}" iyz = "0"
+              izz="${m*r*r/2}" />
+  </macro>
   <link name = 'left_wheel'>
     <visual>
@@ -72,9 +78,5 @@
       <mass value="5.0"/>
       <origin xyz="0 0 0" rpy=" 0 1.5707 1.5707"/>
-      <inertia
-          ixx="0.1" ixy="0" ixz="0"
-          iyy="0.1" iyz="0"
-          izz="0.1"
-      />
+      <cylinder_inertia  m="5.0" r="0.1" h="0.05" />
     </inertial>
   </link>
@@ -95,9 +97,5 @@
       <mass value="5.0"/>
       <origin xyz="0 0 0" rpy=" 0 1.5707 1.5707"/>
-      <inertia
-          ixx="0.1" ixy="0" ixz="0"
-          iyy="0.1" iyz="0"
-          izz="0.1"
-      />
+      <cylinder_inertia  m="5.0" r="0.1" h="0.05" />
     </inertial>
   </link>
